File: hardware/shield_v1.0/FLC100_shield_v1.0.brd (EAGLE design)
At the start: 99.1 x 78.7 mm, 102 parts, among them IC1 MCP3424, IC2 MAX756, IC3 MAX619, IC4 MCP1640, Q1 2N7000, Q2 2N7000, Q3 2N7000, Q4 2N7000, Q5 2N7000, X1 RJ45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

Commit message: Adding files used for first production run.
Parts:
- added C16: 10u, SteveMarple:1206-HAND
- C10, C4: value 100n -> 4u7; device SparkFun:CAP-PTH-SMALL -> SparkFun:CPOL-RADIAL-10UF-25V
- C12: value 220n -> 100n; device SparkFun:CAP-PTH-5MM -> SparkFun:CAP-PTH-SMALL
- C14: value 4u7 -> 220n; device SteveMarple:1206-HAND -> SparkFun:CAP-PTH-5MM
- C15: value 10u -> 4u7
- C2, C9: value 4u7 -> 100n; device SparkFun:CPOL-RADIAL-10UF-25V -> SparkFun:CAP-PTH-SMALL
- C7: value 100u -> 100n; device SparkFun:CPOL-RADIAL-10UF-25V -> SparkFun:CAP-PTH-SMALL
- C8: value 100n -> 100u; device SparkFun:CAP-PTH-SMALL -> SparkFun:CPOL-RADIAL-10UF-25V
- R1, R3, R4, R6: value 4k7 -> 10k
- R10: value 15k -> 910k
- R11: value 510k -> 15k
- R12: value 100k -> 510k; device SteveMarple:RES-AXIAL-0.4 -> SteveMarple:1206-HAND
- R7: value 10k -> 100k
- R8: value 100k -> 10k
- R9: value 910k -> 100k; device SteveMarple:1206-HAND -> SteveMarple:RES-AXIAL-0.4
- U$12: value PAD -> CALUNIUM-SHIELD-V2NO-OUTLINE-NO-HOLES-NO-TEXT; device SteveMarple:PAD -> SteveMarple:CALUNIUM-SHIELD-NO-OUTLINE-NO-HOLES-NO-TEXT-V2
- U$7: value CALUNIUM-SHIELD-V2NO-OUTLINE-NO-HOLES-NO-TEXT -> PAD; device SteveMarple:CALUNIUM-SHIELD-NO-OUTLINE-NO-HOLES-NO-TEXT-V2 -> SteveMarple:PAD
- moved U$30 86.6 mm to (86.4, 57.1), turned to 270 degrees
- moved U$14 85.5 mm to (10.2, 76.2), turned to 0 degrees
- moved U$42 84.4 mm to (12.7, 35.6)
- moved U$15 78.5 mm to (12.7, 76.2), turned to 0 degrees
- moved U$29 77.5 mm to (88.9, 49.5), turned to 270 degrees
- moved U$37 73.6 mm to (78.7, 49.5), turned to 270 degrees
- moved U$13 66.5 mm to (30.5, 30.5), turned to 0 degrees
- moved U$38 66.3 mm to (76.2, 57.1), turned to 270 degrees
- moved C2 64.9 mm to (33.0, 38.1), turned to 270 degrees
- moved R12 62.6 mm to (55.9, 17.8), turned to 90 degrees
- moved C14 59.9 mm to (54.6, 62.2), turned to 90 degrees
- moved U$33 56.6 mm to (83.8, 49.5), turned to 270 degrees
- moved C12 55.7 mm to (90.2, 39.4), turned to 180 degrees
- moved R9 52.1 mm to (36.8, 61.0), turned to 270 degrees
- moved U$36 50.8 mm to (78.7, 57.1), turned to 270 degrees
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Connections:
- net !RESET: now also C12.2, U$12.!RESET@0, U$12.!RESET@1; no longer C11.2, U$7.!RESET@0, U$7.!RESET@1
- net !XRF_RESET: now also U$12.5; no longer U$7.5
- net +3V3: now also C16.1, C5.1, C9.1, R10.2, U$12.3.3V, U$18.1, U$19.1, U$22.1, U$5.1; no longer C15.1, C3.1, C7.1, R9.2, U$36.1, U$42.1, U$43.1, U$7.3.3V, U$9.1
- net +5V: now also C11.1, C2.1, U$21.1; no longer C9.1, U$41.1
- net 0(RX0): now also U$12.0(RX0); no longer U$7.0(RX0)
- net 1(TX0): now also U$12.1(TX0); no longer U$7.1(TX0)
- net 2: now also U$12.2@0; no longer U$7.2@0
- net 20: now also U$12.20@1; no longer U$7.20@1
- net 21: now also U$12.21@1; no longer U$7.21@1
- net 3: now also U$12.3@0; no longer U$7.3@0
- net A4: now also U$12.A4/SDA; no longer U$7.A4/SDA
- net A5: now also U$12.A5/SCL; no longer U$7.A5/SCL
- net A6: now also U$12.A6; no longer U$7.A6
- net A7: now also C7.1, U$12.A7; no longer C6.1, U$7.A7
- net GND: now also C11.2, C16.2, R12.1, R7.P$1, U$12.GND@0, U$12.GND@1, U$12.GND@2, U$12.GND@3, U$14.1, U$15.1, U$16.1, U$17.1; no longer C14.2, R11.1, R12.P$1, U$27.1, U$37.1, U$38.1, U$39.1, U$7.GND@0, U$7.GND@1, U$7.GND@2, U$7.GND@3
- net N$10: now also U$26.1; no longer U$13.1
- net N$11: now also U$28.1; no longer U$15.1
- net N$12: now also U$30.1; no longer U$17.1
- net N$13: now also U$32.1; no longer U$19.1
- net N$14: now also U$34.1; no longer U$21.1
- net N$15: now also U$36.1; no longer U$23.1
- net N$16: now also U$38.1; no longer U$25.1
- net N$17: now also U$27.1; no longer U$14.1
- net N$18: now also C12.1, U$29.1; no longer C11.1, U$16.1
- net N$19: now also U$31.1; no longer U$18.1
- net N$20: now also U$33.1; no longer U$20.1
- net N$21: now also U$35.1; no longer U$22.1
- net N$22: now also U$37.1; no longer U$24.1
- net N$23: now also U$39.1; no longer U$26.1
- net N$24: now also U$41.1; no longer U$28.1
- net N$25: now also U$20.1; no longer U$8.1
- net N$26: now also R7.P$2, U$12.9; no longer R12.P$2, U$7.9
- net N$27: now also U$12.A2; no longer U$7.A2
- net N$28: now also R8.P$1; no longer R7.P$1
- net N$29: now also U$12.5V, U$2.1; no longer U$35.1, U$7.5V
- net N$3: now also C13.2; no longer C12.2
- net N$31: now also C6.1; no longer C5.1
- net N$4: now also C13.1; no longer C12.1
- net N$40: now also U$11.1, U$12.21@0; no longer U$32.1, U$7.21@0
- net N$42: now also R11.1, R12.2; no longer R10.1, R11.2
- net N$43: now also U$12.14, U$3.1; no longer U$1.1, U$7.14
- net N$44: now also U$12.15, U$4.1; no longer U$2.1, U$7.15
- net N$45: now also U$12.16, U$6.1; no longer U$3.1, U$7.16
- net N$46: now also R10.1, R11.2; no longer R10.2, R9.1
- net N$47: now also U$12.17, U$7.1; no longer U$4.1, U$7.17
- net N$48: now also U$12.18, U$8.1; no longer U$5.1, U$7.18
- net N$49: now also U$12.19, U$9.1; no longer U$6.1, U$7.19
- net N$5: now also C14.1; no longer C13.1
- net N$50: now also U$10.1, U$12.20@0; no longer U$31.1, U$7.20@0
- net N$52: now also U$12.IOREF, U$13.1; no longer U$33.1, U$7.IOREF
- net N$6: now also C14.2; no longer C13.2
- net N$7: now also U$23.1; no longer U$10.1
- net N$8: now also U$25.1; no longer U$12.1
- net N$9: now also R8.P$2, U$24.1; no longer R7.P$2, U$11.1
- net SCL_3V3: now also U$12.SCL; no longer U$7.SCL
- net SDA_3V3: now also U$12.SDA; no longer U$7.SDA
- net SHDN: now also R9.P$1; no longer R8.P$1
- net VIN: now also C15.1, C3.1, R9.P$2, U$1.1, U$12.VIN; no longer C14.1, C2.1, R8.P$2, U$34.1, U$7.VIN
- net XRF_SLEEP: now also U$12.7; no longer U$7.7
Routing:
- net GNDZ: track 14.2 -> 0.00 mm
- net VIN: track 175.7 -> 168.4 mm
- net N$31: track 10.7 -> 16.2 mm
- net +3V3: track 261.0 -> 265.6 mm
- net +5V: track 138.2 -> 142.1 mm
- net SCL_5V: track 67.4 -> 68.4 mm
- net SHDN: track 46.0 -> 47.0 mm
- net N$32: track 52.1 -> 53.0 mm
- net GND: track 435.7 -> 435.0 mm
Other:
- board text added: ">PLOT_DATE_TIME"
- board text removed: ">LAST_DATE_TIME"
