File: hardware/shield_v1.0/FLC100_shield_v1.0.sch (EAGLE design)
At the start: 102 parts, among them IC1 MCP3424, IC2 MAX756, IC3 MAX619, IC4 MCP1640, Q1 2N7000, Q2 2N7000, Q3 2N7000, Q4 2N7000, Q5 2N7000, X1 RJ45, X2 RJ45

Commit message: Adding files used for first production run.
Parts:
- added C16: 10u, SteveMarple:C-EU1206-HAND
- C10, C4: value 100n -> 4u7; device SparkFun:CAPPTH -> SparkFun:CAP_POLPTH2
- C12: value 220n -> 100n; device SparkFun:CAPPTH1 -> SparkFun:CAPPTH
- C14: value 4u7 -> 220n; device SteveMarple:C-EU1206-HAND -> SparkFun:CAPPTH1
- C15: value 10u -> 4u7
- C2, C9: value 4u7 -> 100n; device SparkFun:CAP_POLPTH2 -> SparkFun:CAPPTH
- C7: value 100u -> 100n; device SparkFun:CAP_POLPTH2 -> SparkFun:CAPPTH
- C8: value 100n -> 100u; device SparkFun:CAPPTH -> SparkFun:CAP_POLPTH2
- R1, R3, R4, R6: value 4k7 -> 10k
- R10: value 15k -> 910k
- R11: value 510k -> 15k
- R12: value 100k -> 510k; device SteveMarple:RESISTOR -> SteveMarple:RESISTOR1206-HAND
- R7: value 10k -> 100k
- R8: value 100k -> 10k
- R9: value 910k -> 100k; device SteveMarple:RESISTOR1206-HAND -> SteveMarple:RESISTOR
- U$12: value PAD -> CALUNIUM-SHIELD-V2NO-OUTLINE-NO-HOLES-NO-TEXT; device SteveMarple:PAD -> SteveMarple:CALUNIUM-SHIELD-V2NO-OUTLINE-NO-HOLES-NO-TEXT
- U$7: value CALUNIUM-SHIELD-V2NO-OUTLINE-NO-HOLES-NO-TEXT -> PAD; device SteveMarple:CALUNIUM-SHIELD-V2NO-OUTLINE-NO-HOLES-NO-TEXT -> SteveMarple:PAD
Connections:
- net !RESET: now also C12.2, U$12.!RESET@0, U$12.!RESET@1; no longer C11.2, U$7.!RESET@0, U$7.!RESET@1
- net !XRF_RESET: now also U$12.5; no longer U$7.5
- net +3V3: now also C16.1, C4.+, C5.1, C8.+, C9.1, R10.2, U$12.3.3V, U$18.1, U$19.1, U$22.1, U$5.1; no longer C15.1, C3.+, C4.1, C7.+, C8.1, R9.2, U$36.1, U$42.1, U$43.1, U$7.3.3V, U$9.1
- net +5V: now also C10.+, C11.1, C2.1, U$21.1; no longer C10.1, C9.+, U$41.1
- net 0(RX0): now also U$12.0(RX0); no longer U$7.0(RX0)
- net 1(TX0): now also U$12.1(TX0); no longer U$7.1(TX0)
- net 2: now also U$12.2(RX1)@0; no longer U$7.2(RX1)@0
- net 20: now also U$12.20(SDA)@1; no longer U$7.20(SDA)@1
- net 21: now also U$12.21(SCL)@1; no longer U$7.21(SCL)@1
- net 3: now also U$12.3(TX1)@0; no longer U$7.3(TX1)@0
- net A4: now also U$12.A4; no longer U$7.A4
- net A5: now also U$12.A5; no longer U$7.A5
- net A6: now also U$12.A6; no longer U$7.A6
- net A7: now also C7.1, U$12.A7; no longer C6.1, U$7.A7
- net GND: now also C10.-, C11.2, C16.2, C2.2, C4.-, C7.2, C8.-, C9.2, R7.1, U$12.GND@0, U$12.GND@1, U$12.GND@2, U$12.GND@3, U$14.1, U$15.1, U$16.1, U$17.1; no longer C10.2, C14.2, C2.-, C4.2, C7.-, C8.2, C9.-, R11.1, U$27.1, U$37.1, U$38.1, U$39.1, U$7.GND@0, U$7.GND@1, U$7.GND@2, U$7.GND@3
- net N$10: now also U$26.1; no longer U$13.1
- net N$11: now also U$28.1; no longer U$15.1
- net N$12: now also U$30.1; no longer U$17.1
- net N$13: now also U$32.1; no longer U$19.1
- net N$14: now also U$34.1; no longer U$21.1
- net N$15: now also U$36.1; no longer U$23.1
- net N$16: now also U$38.1; no longer U$25.1
- net N$17: now also U$27.1; no longer U$14.1
- net N$18: now also C12.1, U$29.1; no longer C11.1, U$16.1
- net N$19: now also U$31.1; no longer U$18.1
- net N$20: now also U$33.1; no longer U$20.1
- net N$21: now also U$35.1; no longer U$22.1
- net N$22: now also U$37.1; no longer U$24.1
- net N$23: now also U$39.1; no longer U$26.1
- net N$24: now also U$41.1; no longer U$28.1
- net N$25: now also U$20.1; no longer U$8.1
- net N$26: now also R7.2, U$12.9; no longer R12.2, U$7.9
- net N$27: now also U$12.A2; no longer U$7.A2
- net N$28: now also R8.1; no longer R7.1
- net N$29: now also U$12.5V, U$2.1; no longer U$35.1, U$7.5V
- net N$3: now also C13.2; no longer C12.2
- net N$31: now also C6.1; no longer C5.1
- net N$4: now also C13.1; no longer C12.1
- net N$40: now also U$11.1, U$12.21(SCL)@0; no longer U$32.1, U$7.21(SCL)@0
- net N$42: now also R11.1, R12.2; no longer R10.1, R11.2
- net N$43: now also U$12.14, U$3.1; no longer U$1.1, U$7.14
- net N$44: now also U$12.15, U$4.1; no longer U$2.1, U$7.15
- net N$45: now also U$12.16, U$6.1; no longer U$3.1, U$7.16
- net N$46: now also R10.1, R11.2; no longer R10.2, R9.1
- net N$47: now also U$12.17, U$7.1; no longer U$4.1, U$7.17
- net N$48: now also U$12.18, U$8.1; no longer U$5.1, U$7.18
- net N$49: now also U$12.19, U$9.1; no longer U$6.1, U$7.19
- net N$5: now also C14.1; no longer C13.1
- net N$50: now also U$10.1, U$12.20(SDA)@0; no longer U$31.1, U$7.20(SDA)@0
- net N$52: now also U$12.IOREF, U$13.1; no longer U$33.1, U$7.IOREF
- net N$6: now also C14.2; no longer C13.2
- net N$7: now also U$23.1; no longer U$10.1
- net N$8: now also U$25.1; no longer U$12.1
- net N$9: now also R8.2, U$24.1; no longer R7.2, U$11.1
- net SCL_3V3: now also U$12.SCL; no longer U$7.SCL
- net SDA_3V3: now also U$12.SDA; no longer U$7.SDA
- net SHDN: now also R9.1; no longer R8.1
- net VIN: now also C15.1, C3.+, R9.2, U$1.1, U$12.VIN; no longer C14.1, C2.+, R8.2, U$34.1, U$7.VIN
- net XRF_SLEEP: now also U$12.7; no longer U$7.7
Other:
- note removed: "Check !SHDN! and 3/!5! pins"
- note removed: "Check connectors from Calunium"
- moved on the sheet: C1, C11, C12, C13, C14, C15, C3, C5, C6, R10, R11, R12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
